File: 0028_Button_Module_Tact.kicad_sch (KiCad schematic)
At the start: 5 parts

Commit message: Add files via upload
Parts:
- added D2, D3, D4: LED, LED_SMD:LED_0603_1608Metric, symbol Device:LED
- added R10: 470r, Resistor_SMD:R_0603_1608Metric, symbol Device:R
- added R4, R6, R7, R9: 1k, Resistor_SMD:R_0603_1608Metric, symbol Device:R
- added R5, R8: 10k, Resistor_SMD:R_0603_1608Metric, symbol Device:R
- added S2, S3: B3F-5050, meminle:B3F-4055, symbol B3F-5050:B3F-5050
- added U1: ~, Moduler_:pin_header_5-3, symbol moduler_pin:air
- D1: footprint (none) -> LED_SMD:LED_0603_1608Metric
- R1, R2, R3: footprint (none) -> Resistor_SMD:R_0603_1608Metric
- S1: footprint B3F-4055 -> meminle:B3F-4055
Connections:
- net GND: now also D2.1 (K), D3.1 (K), D4.1 (K), R5.2, R8.2, U1.9
- net SIG renamed SIG1
- net SIG1: now also U1.12
- net VCC renamed +3V3
- net +3V3: now also R10.1, S2.1 (COM_1), S2.3 (NO_1), S3.1 (COM_1), S3.3 (NO_1), U1.8
- new net: R7.1, R8.1, R9.1, S3.2 (COM_2), S3.4 (NO_2)
- new net: R4.1, R5.1, R6.1, S2.2 (COM_2), S2.4 (NO_2)
- new net: D2.2 (A), R4.2
- new net: D3.2 (A), R7.2
- new net: D4.2 (A), R10.2
- new net SIG2: R6.2, U1.13
- new net SIG3: R9.2, U1.14
- no-connect marks 0 -> 13
Other:
- note added: "AIR PIN"
- note added: "SENSOR"
- moved on the sheet: D1, R1, R2, R3, S1
